File: msv-pcb/msv-pcb.kicad_sch (KiCad schematic)
At the start: 0 parts

Commit message: Power Circuit Done
Parts:
- added BT1: Battery_Cell, symbol Device:Battery_Cell
- added C1: 1µF, symbol Device:C
- added C2: 100µF, symbol Device:C
- added PN1: ~, symbol msv-pcb-utils:PN532 Module V3
- added U1: ~, symbol msv-pcb-utils:TP4056_Charging_Module_Type_C
- added U2: ESP-07, RF_Module:ESP-07, symbol RF_Module:ESP-07
- added VR1: MCP1700T-3302E_MB(SOT89-3), OLIMEX_Regulators-FP:SOT89-3, symbol OLIMEX_Regulators:MCP1700T-3302E_MB(SOT89-3)
Connections:
- new net: C1.1, U1.6 (B-), VR1.2 (VIN)
- new net: BT1.1 (+), U1.4 (OUT-)
- new net: BT1.2 (-), U1.6 (B-)
- new net GND: C1.2, C2.2, U1.4 (OUT-), VR1.1 (GND)
- new net VCC: C2.1, VR1.3 (VOUT)
Other:
- note added: "POWER CIRCUIT"

Commit message: Circuit schematics
Parts:
- removed BT1: Battery_Cell, symbol Device:Battery_Cell
- added J1: Conn_01x02_Pin, Connector_PinHeader_1.27mm:PinHeader_1x02_P1.27mm_Vertical, symbol Connector:Conn_01x02_Pin
- added J2: Conn_01x05_Socket, symbol Connector:Conn_01x05_Socket
- added R1, R2: 45K, symbol Device:R
- added R3, R4: 10K, symbol Device:R
- added R5: 30K, symbol Device:R
- added U3: ULN2003, symbol Transistor_Array:ULN2003
Connections:
- net GND: now also PN1.12 (GND), U1.3 (B-), U2.9 (GND), J2.5 (Pin_5), R5.1, U3.8 (GND)
- net VCC: now also PN1.11 (VCC), U2.8 (VCC), R1.1, R2.1, R3.1, R4.1
- net RST: now reaches U2.1 (~{RST})
- net RST: now also R4.2
- net GPIO 15: now reaches U2.10 (GPIO15)
- net GPIO 15: now also R5.2
- net GPIO 2: now reaches U2.11 (GPIO2)
- net GPIO 2: now also R2.2
- net GPIO 0: now reaches U2.12 (GPIO0)
- net GPIO 0: now also R1.2
- net PHASE A: now reaches U2.13 (GPIO4)
- net PHASE A: now also U3.1 (I1)
- net PHASE B: now reaches U2.14 (GPIO5)
- net PHASE B: now also U3.2 (I2)
- net RXD: now reaches U2.15 (GPIO3/RXD)
- net RXD: now also J1.2 (Pin_2)
- net TXD: now reaches U2.16 (GPIO1/TXD)
- net TXD: now also J1.1 (Pin_1)
- net EN: now reaches U2.3 (EN)
- net EN: now also R3.2
- net IC2 1: now reaches U2.4 (GPIO16)
- net IC2 1: now also PN1.10 (SDA)
- net IC2 2: now reaches U2.5 (GPIO14)
- net IC2 2: now also PN1.9 (SCL)
- net PHASE C: now reaches U2.6 (GPIO12)
- net PHASE C: now also U3.3 (I3)
- net PHASE D: now reaches U2.7 (GPIO13)
- net PHASE D: now also U3.4 (I4)
- net 5v: now reaches C1.1, VR1.2 (VIN)
- net 5v: now also U1.1 (OUT_+), U3.9 (COM); no longer U1.6 (B-)
- new net: J2.4 (Pin_4), U3.13 (O4)
- new net: J2.3 (Pin_3), U3.14 (O3)
- new net: J2.2 (Pin_2), U3.15 (O2)
- new net: J2.1 (Pin_1), U3.16 (O1)
- new net +5V: U1.2 (B+)
- no-connect marks 0 -> 17
Other:
- note added: "DEBUG"
- note added: "PULL UP/DOWN NETWORK"
- moved on the sheet: PN1, U2

Commit message: Started footprint assosiations
Parts:
- C1, C2: footprint (none) -> Capacitor_SMD:C_0805_2012Metric_Pad1.18x1.45mm_HandSolder
- J2: footprint (none) -> Connector_JST:JST_XH_B5B-XH-AM_1x05_P2.50mm_Vertical
- R1, R2, R3, R4, R5: footprint (none) -> Resistor_SMD:R_0805_2012Metric_Pad1.20x1.40mm_HandSolder
- U3: footprint (none) -> Package_DIP:DIP-16_W7.62mm_Socket_LongPads
Changed lines of the file:
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@@
 			)
 		)
-		(property "Footprint" ""
+		(property "Footprint" "Resistor_SMD:R_0805_2012Metric_Pad1.20x1.40mm_HandSolder"
 			(at 156.21 183.388 90)
 			(effects
@@
 			)
 		)
-		(property "Footprint" ""
+		(property "Footprint" "Resistor_SMD:R_0805_2012Metric_Pad1.20x1.40mm_HandSolder"
 			(at 156.21 152.908 90)
 			(effects
@@
 			)
 		)
-		(property "Footprint" ""
+		(property "Footprint" "Capacitor_SMD:C_0805_2012Metric_Pad1.18x1.45mm_HandSolder"
 			(at 77.1652 181.61 0)
 			(effects
@@
 			)
 		)
-		(property "Footprint" ""
+		(property "Footprint" "Resistor_SMD:R_0805_2012Metric_Pad1.20x1.40mm_HandSolder"
 			(at 156.21 163.068 90)
 			(effects
@@
 			)
 		)
-		(property "Footprint" ""
+		(property "Footprint" "Resistor_SMD:R_0805_2012Metric_Pad1.20x1.40mm_HandSolder"
 			(at 134.62 149.352 90)
 			(effects
@@
 			)
 		)
-		(property "Footprint" ""
+		(property "Footprint" "Package_DIP:DIP-16_W7.62mm_Socket_LongPads"
 			(at 199.39 107.95 0)
 			(effects
@@
 			)
 		)
-		(property "Footprint" ""
+		(property "Footprint" "Resistor_SMD:R_0805_2012Metric_Pad1.20x1.40mm_HandSolder"
 			(at 156.21 173.228 90)
 			(effects
@@
 			)
 		)
-		(property "Footprint" ""
+		(property "Footprint" "Capacitor_SMD:C_0805_2012Metric_Pad1.18x1.45mm_HandSolder"
 			(at 97.4852 181.61 0)
 			(effects
@@
 			)
 		)
-		(property "Footprint" ""
+		(property "Footprint" "Connector_JST:JST_XH_B5B-XH-AM_1x05_P2.50mm_Vertical"
 			(at 222.25 93.98 0)
 			(effects
